Commit message: replan step1 test in v1, todo change the error in 217line, get the diff curve with diff goals

File: ur3e.urdf (robot description, URDF)
Before this commit: robot ur3, 9 links, 8 joints
Links:
- added link tool_mid
Joints:
- removed joint wrist_3_link-tool0_fixed_joint
- added joint tool_mid-tool0_fixed_joint: type fixed, parent tool_mid, child tool0, origin xyz=-0.1117 0.20432 0 rpy=-1.57079632679 0 0
- added joint wrist_3_link-toolmid_fixed_joint: type fixed, parent wrist_3_link, child tool_mid, origin xyz=0 0 0 rpy=0 0.7853982 0

Commit message: replan v1 update, depart to 3 phase and complete the demo

File: ur3e.urdf (robot description, URDF)
Before this commit: robot ur3, 10 links, 9 joints
Joints:
- joint tool_mid-tool0_fixed_joint: origin xyz=-0.1117 0.20432 0 rpy=-1.57079632679 0 0 -> xyz=-0.142 0.20045 0 rpy=-1.57079632679 0 0
